File: kicad/stm32f103c8t6-qwiic.kicad_pcb (KiCad board)
At the start: 2 copper layers, 58.4 x 22.7 mm, 39 parts, among them J1 Conn_01x04_Pin, J2 Conn_01x04_Pin, J3 Conn_01x04_Pin, J4 Conn_01x16_Pin, J5 Conn_01x16_Pin, J6 USB_C_USB2.0_14P, SW1 SW_Push, SW2 SW_Push, U1 STM32F103C8Tx, U2 ME6211C33M5G-N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

Commit message: Update KiCAD files due to wrong footprint BM04B was chosen instead of SM04B for the Qwiic connectors. This commit updates the footprints, layout and production files.
Parts:
- J1, J2, J3: footprint Connector_JST:JST_SH_BM04B-SRSS-TB_1x04-1MP_P1.00mm_Vertical -> Connector_JST:JST_SH_SM04B-SRSS-TB_1x04-1MP_P1.00mm_Horizontal
- moved J1 0.70 mm to (72.1, 28.8), turned to 90 degrees
- moved J2 0.70 mm to (69.5, 36.8), turned to 0 degrees
- moved J3 0.70 mm to (69.5, 20.7), turned to 180 degrees
Routing:
- net /I2C1_SCL: track 36.2 -> 40.1 mm
- net /BOOT: track 23.7 -> 27.0 mm
- net /SWCLK: track 30.4 -> 33.3 mm
- net /SWDIO: track 31.2 -> 32.2 mm
- net /I2C2_SCL: track 33.7 -> 32.7 mm
- net +3.3V: track 122.3 -> 121.6 mm
- net GND: track 48.4 -> 47.7 mm, vias 41 -> 40
