File: kicad/stm32f103c8t6-qwiic.kicad_sch (KiCad schematic)
At the start: 39 parts, among them J1 Conn_01x04_Pin, J2 Conn_01x04_Pin, J3 Conn_01x04_Pin, J4 Conn_01x16_Pin, J5 Conn_01x16_Pin, J6 USB_C_USB2.0_14P, SW1 SW_Push, SW2 SW_Push, U1 STM32F103C8Tx, U2 ME6211C33M5G-N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

Commit message: Update KiCAD files due to wrong footprint BM04B was chosen instead of SM04B for the Qwiic connectors. This commit updates the footprints, layout and production files.
Parts:
- J1, J2, J3: footprint Connector_JST:JST_SH_BM04B-SRSS-TB_1x04-1MP_P1.00mm_Vertical -> Connector_JST:JST_SH_SM04B-SRSS-TB_1x04-1MP_P1.00mm_Horizontal
Changed lines of the file:
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@@
 			)
 		)
-		(property "Footprint" "Connector_JST:JST_SH_BM04B-SRSS-TB_1x04-1MP_P1.00mm_Vertical"
+		(property "Footprint" "Connector_JST:JST_SH_SM04B-SRSS-TB_1x04-1MP_P1.00mm_Horizontal"
 			(at 264.16 114.3 0)
 			(effects
@@
 			)
 		)
-		(property "Footprint" "Connector_JST:JST_SH_BM04B-SRSS-TB_1x04-1MP_P1.00mm_Vertical"
+		(property "Footprint" "Connector_JST:JST_SH_SM04B-SRSS-TB_1x04-1MP_P1.00mm_Horizontal"
 			(at 217.17 114.3 0)
 			(effects
@@
 			)
 		)
-		(property "Footprint" "Connector_JST:JST_SH_BM04B-SRSS-TB_1x04-1MP_P1.00mm_Vertical"
+		(property "Footprint" "Connector_JST:JST_SH_SM04B-SRSS-TB_1x04-1MP_P1.00mm_Horizontal"
 			(at 241.3 114.3 0)
 			(effects
